Commit message: Updated obstacle

File: src/Hector_Simulation-ROS_Simulation/Hector_ROS_Simulation/hector_description/xacro/const.xacro (robot description, xacro)
@@ -217,3 +217,16 @@
     <xacro:property name="toe_iyz" value="0.0"/>
     <xacro:property name="toe_izz" value="0.0002"/>
+    <!-- SLAMTECH LiDAR (M2M2) Properties -->
+    <xacro:property name="lidar_mass" value="0.165"/>
+    <xacro:property name="lidar_length" value="0.0749"/>
+    <xacro:property name="lidar_radius" value="0.03855"/>
+    <xacro:property name="lidar_com_x" value="0.0"/>
+    <xacro:property name="lidar_com_y" value="0.0"/>
+    <xacro:property name="lidar_com_z" value="0.0"/>
+    <xacro:property name="lidar_ixx" value="0.001"/>
+    <xacro:property name="lidar_ixy" value="0.0"/>
+    <xacro:property name="lidar_ixz" value="0.0"/>
+    <xacro:property name="lidar_iyy" value="0.001"/>
+    <xacro:property name="lidar_iyz" value="0.0"/>
+    <xacro:property name="lidar_izz" value="0.001"/>
 </robot>

File: src/Hector_Simulation-ROS_Simulation/Hector_ROS_Simulation/hector_description/xacro/gazebo.xacro (robot description, xacro)
@@ -145,3 +145,30 @@
         <material>Gazebo/Grey</material>
     </gazebo>
+    <!-- Lidar Sensor Plugin -->
+    <gazebo reference="lidar_link">
+        <sensor type="ray" name="lidar_sensor">
+            <update_rate>10</update_rate> <!-- Adjust if necessary -->
+            <pose>0 0 0 0 0 0</pose>
+            <visualize>true</visualize>
+            <ray>
+                <scan>
+                    <horizontal>
+                        <samples>360</samples>
+                        <resolution>0.391</resolution>
+                        <min_angle>-3.1415</min_angle>
+                        <max_angle>3.1415</max_angle>
+                    </horizontal>
+                </scan>
+                <range>
+                    <min>0.1</min>
+                    <max>40.0</max> <!-- Adjust based on lidar specs -->
+                    <resolution>0.03</resolution>
+                </range>
+            </ray>
+            <plugin name="gazebo_ros_laser_controller" filename="libgazebo_ros_laser.so">
+                <topicName>/scan</topicName>
+                <frameName>lidar_link</frameName>
+            </plugin>
+        </sensor>
+    </gazebo>
 </robot>

File: src/Hector_Simulation-ROS_Simulation/Hector_ROS_Simulation/hector_description/xacro/materials.xacro (robot description, xacro)
@@ -28,3 +28,6 @@
         <color rgba="1.0 1.0 1.0 1.0"/>
     </material>
+    <material name="lidar_grey">
+        <color rgba="0.5 0.5 0.5 1.0"/>
+    </material>
 </robot>

File: src/Hector_Simulation-ROS_Simulation/Hector_ROS_Simulation/hector_description/xacro/robot.xacro (robot description, xacro)
@@ -1,4 +1,5 @@
 <?xml version="1.0"?>
 <robot name="hector_description" xmlns:xacro="http://www.ros.org/wiki/xacro">
+    <!--link name="world"/-->
     <xacro:include filename="$(find hector_description)/xacro/const.xacro"/>
     <xacro:include filename="$(find hector_description)/xacro/materials.xacro"/>
@@ -18,4 +19,9 @@
         </joint>
     </xacro:if>
+    <!--joint name="world_to_base" type="fixed">
+        <origin rpy="0 0 0" xyz="0 0 0"/>
+        <parent link="world"/>
+        <child link="base"/>
+    </joint-->
     <link name="base">
         <visual>
@@ -114,3 +120,57 @@
         <origin rpy="0 0 0" xyz="${hip_offset_x} ${-hip_offset_y} ${-hip_offset_z}"/>
     </xacro:leg>
+    <!-- LiDAR link and joint -->
+    <link name="lidar_link">
+        <inertial>
+            <origin rpy="0 0 0" xyz="${lidar_com_x} ${lidar_com_y} ${lidar_com_z}"/>
+            <mass value="${lidar_mass}"/>
+            <inertia ixx="${lidar_ixx}" ixy="${lidar_ixy}" ixz="${lidar_ixz}" iyy="${lidar_iyy}" iyz="${lidar_iyz}" izz="${lidar_izz}"/>
+        </inertial>
+        <visual>
+            <origin rpy="0 0 0" xyz="0 0 0"/>
+            <geometry>
+                <cylinder length="${lidar_length}" radius="${lidar_radius}"/>
+            </geometry>
+            <material name="grey"/>
+        </visual>
+        <collision>
+            <origin rpy="0 0 0" xyz="0 0 0"/>
+            <geometry>
+                <cylinder length="${lidar_length}" radius="${lidar_radius}"/>
+            </geometry>
+        </collision>
+    </link>
+    <!-- Joint to attach the LiDAR to the trunk-->
+    <joint name="lidar_joint" type="fixed">
+        <parent link="trunk"/>
+        <child link="lidar_link"/>
+        <origin rpy="0 0 0" xyz="0.0 0.0 0.17"/>
+    </joint>
+     <!-- Temporary Obstacle link and joint to test LiDAR-->
+    <!--link name="obstacle">
+        <visual>
+            <origin rpy="0 0 0" xyz="1.0 0.0 0.0"/>
+            <geometry>
+                <box size="0.5 0.5 0.5"/>
+            </geometry>
+            <material name="blue"/>
+        </visual>
+        <collision>
+            <origin rpy="0 0 0" xyz="1.0 0.0 0.0"/>
+            <geometry>
+                <box size="0.5 0.5 0.5"/>
+            </geometry>
+        </collision>
+        <inertial>
+            <mass value="10.0"/>
+            <origin xyz="0 0 0" rpy="0 0 0"/>
+            <inertia ixx="0.1" ixy="0.0" ixz="0.0" iyy="0.1" iyz="0.0" izz="0.1"/>
+        </inertial>
+    </link-->
+    <!--Joint to attach the LiDAR to the trunk-->
+    <!--joint name="obstacle_fixed_joint" type="fixed">
+        <parent link="world"/>
+        <child link="obstacle"/>
+        <origin rpy="0 0 0" xyz="5.0 0.0 0.0"/>
+    </joint-->
 </robot>
